File: wingcam_ee/mpu.kicad_sch (KiCad schematic)
At the start: 14 parts, among them U1 RV1103G

Commit message: Schematic finished
Parts:
- added C32, C38: 10pF, Capacitor_SMD:C_0402_1005Metric, symbol Device:C_Small
- added D1, D2: LED, LED_SMD:LED_0402_1005Metric, symbol Device:LED
- added R11, R12: 4.7k, Resistor_SMD:R_0402_1005Metric, symbol Device:R_Small
- added R16, R19: 22R, Resistor_SMD:R_0402_1005Metric, symbol Device:R_Small
- added R17, R18: 10k, Resistor_SMD:R_0402_1005Metric, symbol Device:R_Small
- added R20: 1M, Resistor_SMD:R_0402_1005Metric, symbol Device:R_Small
- added R23, R24: 1k, Resistor_SMD:R_0402_1005Metric, symbol Device:R_Small
- added R25: 6.04k, Resistor_SMD:R_0402_1005Metric, symbol Device:R_Small
- added TP1, TP2: TestPoint, TestPoint:TestPoint_Pad_1.5x1.5mm, symbol Connector:TestPoint
- added Y2: 24Mhz, Crystal:Crystal_SMD_2016-4Pin_2.0x1.6mm, symbol Device:Crystal_GND24
- C17, C18, C19, C20, C21, C22, C23, C24, C25, C26, C27, C28: footprint (none) -> Capacitor_SMD:C_0402_1005Metric
- R10: footprint (none) -> Resistor_SMD:R_0402_1005Metric
Connections:
- net +1V8: now also U1.59 (VCCIO6_VCC), R11.1, R12.1
- net +3V3: now also R17.1, R18.1; no longer U1.59 (VCCIO6_VCC)
- net GND: now also C32.2, C38.1, R23.2, R24.2, R25.1, Y2.2 (G), Y2.4 (G)
- net FSPI.D3: now reaches U1.28 (FSPI_D3)
- net FSPI.D3: now also R18.2
- net FSPI.D0: now reaches U1.29 (FSPI_D0)
- net FSPI.D1: now reaches U1.30 (FSPI_D1)
- net FSPI.D2: now reaches U1.31 (FSPI_D2)
- net FSPI.D2: now also R17.2
- net FSPI.~{CS}: now reaches U1.32 (FSPI_CS0)
- net at U1.33 (FSPI_CLK): now also R16.1
- net EPHY.RXN: now reaches U1.67 (FEPHY_RXN)
- net EPHY.RXP: now reaches U1.68 (FEPHY_RXP)
- net EPHY.TXN: now reaches U1.69 (FEPHY_TXN)
- net EPHY.TXP: now reaches U1.70 (FEPHY_TXP)
- net at U1.72 (FEPHY_EXTR): now also R25.2
- net USB.DN: now reaches U1.18 (USB_DM)
- net USB.DP: now reaches U1.19 (USB_DP)
- net at U1.45 (OSC_SOC_XIN): now also C32.1, R20.2, Y2.1
- net at U1.46 (OSC_SOC_XOUT): now also R19.2, R20.1
- net UART_RX: now reaches U1.49 (JTAG_CPU_TCK_M1)
- net UART_RX: now also TP2.1
- net UART_TX: now reaches U1.50 (JTAG_CPU_TMS_M1)
- net UART_TX: now also TP1.1
- net LED2: now reaches U1.53 (PWM11_IR_M1)
- net LED2: now also D2.2 (A)
- net I2C3.SCL: now reaches U1.54 (I2C3_SCL_M1)
- net I2C3.SDA: now reaches U1.55 (I2C3_SDA_M1)
- net LED1: now reaches U1.56 (PWM10_M2)
- net LED1: now also D1.2 (A)
- net STROBE1: now reaches U1.60 (PWM9_M1)
- net VSYNC1: now reaches U1.61 (PWM8_M1)
- net I2C4.SDA: now reaches U1.62 (PWM6_M2)
- net I2C4.SDA: now also R12.2
- net I2C4.SCL: now reaches U1.63 (PWM5_M2)
- net I2C4.SCL: now also R11.2
- net XSHUTDOWN1: now reaches U1.64 (PWM4_M2)
- net CK0N renamed MIPI1.CK0N
- net CK0P renamed MIPI1.CK0P
- net CK1N renamed MIPI2.CK0N
- net CK1P renamed MIPI2.CK0P
- net CLK0: no longer names the net of U1.1 (MIPI_CLK0_OUT)
- net D0N renamed MIPI1.D0N
- net D0P renamed MIPI1.D0P
- net D1N renamed MIPI1.D1N
- net D1P renamed MIPI1.D1P
- net D2N renamed MIPI2.D0N
- net D2P renamed MIPI2.D0P
- net D3N renamed MIPI2.D1N
- net D3P renamed MIPI2.D1P
- net MMC1.CLK renamed SDMMC.CLK
- net MMC1.CMD renamed SDMMC.CMD
- net MMC1.DAT0 renamed SDMMC.D0
- net MMC1.DAT1 renamed SDMMC.D1
- net MMC1.DAT2 renamed SDMMC.D2
- net MMC1.DAT3 renamed SDMMC.D3
- net MMC1.DET renamed SDMMC.DET
- new net: D2.1 (K), R24.1
- new net: C38.2, R19.1, Y2.3
- new net: D1.1 (K), R23.1
- new net FSPI.CLK: R16.2
- no-connect marks 0 -> 5
Other:
- note added: "Pins 62/63 I2C4_M1 -> VCCIO6_VCC domain -> 1.8V Pins 54/55 I2C3_M1 -> VCCIO1_VCC3V3 domain Pins 4/5 I2C4_M2 -> GPIO3_VCC domain"
