File: wingcam_ee/pmic.kicad_sch (KiCad schematic)
At the start: 29 parts, among them U2 EA3036C

Commit message: Schematic finished
Parts:
- added C29, C30, C33, C34: 1uF, Capacitor_SMD:C_0402_1005Metric, symbol Device:C_Small
- added U4: TLV73312PDBV, Package_TO_SOT_SMD:SOT-23-5, symbol Regulator_Linear:TLV73312PDBV
- added U6: TLV73328PDBV, Package_TO_SOT_SMD:SOT-23-5, symbol Regulator_Linear:TLV73328PDBV
- C1, C10, C11, C12, C13, C14, C15, C16, C2, C3, C4, C5, C6, C7, C8, C9: footprint (none) -> Capacitor_SMD:C_0402_1005Metric
- R1, R2, R3, R4, R5, R6, R7, R8, R9: footprint (none) -> Resistor_SMD:R_0402_1005Metric
- U2: footprint Package_DFN_QFN:QFN-20-1EP_3x3mm_P0.45mm_EP1.6x1.6mm -> Package_DFN_QFN:QFN-20-1EP_3x3mm_P0.4mm_EP1.65x1.65mm
Connections:
- net +3V3: now also C29.1, C33.1, U4.1 (IN), U4.3 (EN), U6.1 (IN), U6.3 (EN)
- net GND: now also C29.2, C30.2, C33.2, C34.2, U4.2 (GND), U6.2 (GND)
- new net +1V2: C30.1, U4.5 (OUT)
- new net +2V8: C34.1, U6.5 (OUT)
Other:
- moved on the sheet: C1, C10, C11, C12, C13, C14, C15, C16, C2, C3, C4, C5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
