File: wingcam_ee/wingcam_ee.kicad_sch (KiCad schematic)
At the start: 2 parts, among them J1 Micro_SD_Card_Det1, P1 USB_C_Plug_USB2.0

Commit message: Schematic finished
Parts:
- removed J1: Micro_SD_Card_Det1, symbol Connector:Micro_SD_Card_Det1
- removed P1: USB_C_Plug_USB2.0, symbol Connector:USB_C_Plug_USB2.0
- added C50: 10uF, Capacitor_SMD:C_0402_1005Metric, symbol Device:C_Small
- added H1, H2, H3, H4: M2, MountingHole:MountingHole_2.2mm_M2, symbol Mechanical:MountingHole
- added J1: USB_C_Receptacle_USB2.0_16P, Connector_USB:USB_C_Receptacle_GCT_USB4105-xx-A_16P_TopMnt_Horizontal, symbol Connector:USB_C_Receptacle_USB2.0_16P
- added J2: Micro_SD_Card_Det2, Connector_Card:microSD_HC_Hirose_DM3AT-SF-PEJM5, symbol Connector:Micro_SD_Card_Det2
- added J3: RJ45_Hanrun_HR911105A_Horizontal, Connector_RJ:RJ45_Hanrun_HR911105A_Horizontal, symbol Connector:RJ45_Hanrun_HR911105A_Horizontal
- added J4: JST, Connector_JST:JST_SH_SM04B-SRSS-TB_1x04-1MP_P1.00mm_Horizontal, symbol Connector:Conn_01x04_Pin
- added MP1, MP2: Camera_Lens_20mm, ov9281:Camera_Lens_20mm, symbol wingcam:Camera_Lens_20mm
- added R14, R15: 5.6k, Resistor_SMD:R_0402_1005Metric, symbol Device:R_Small
- added R26, R27, R28, R29: 49.9R, Resistor_SMD:R_0402_1005Metric, symbol Device:R_Small
- added R30, R31: 330R, Resistor_SMD:R_0402_1005Metric, symbol Device:R_Small
- added RN1, RN2: 47k, Resistor_SMD:R_Array_Concave_4x0402, symbol Device:R_Pack04
- added U5: TPD2EUSB30, Package_TO_SOT_SMD:Texas_DRT-3, symbol Power_Protection:TPD2EUSB30
Connections:
- net +5V: now also J1.A4 (VBUS), J1.A9 (VBUS), J1.B4 (VBUS), J1.B9 (VBUS), J4.1 (Pin_1)
- net GND: now also C50.2, J1.A1 (GND), J1.A12 (GND), J1.B1 (GND), J1.B12 (GND), J1.SH (SHIELD), J2.6 (VSS), J2.SH (SHIELD), J3.8, J3.SH, J4.4 (Pin_4), R14.1, R15.2, U5.3 (GND)
- new net: J2.10 (DET_A), RN2.2 (R2.1)
- new net: J1.A5 (CC1), R14.2
- new net: J3.10, R31.2
- new net: J3.11, R30.2
- new net: J1.B5 (CC2), R15.1
- new net +3V3: C50.1, J2.4 (VDD), J3.12, J3.4 (TCT), J3.5 (RCT), J3.9, R26.2, R27.2, R28.2, R29.2, RN1.5 (R4.2), RN1.6 (R3.2), RN1.7 (R2.2), RN1.8 (R1.2), RN2.5 (R4.2), RN2.6 (R3.2), RN2.7 (R2.2), RN2.8 (R1.2)
- new net EPHY.RXN: J3.6 (RD-), R28.1
- new net EPHY.RXP: J3.3 (RD+), R29.1
- new net EPHY.TXN: J3.2 (TD-), R27.1
- new net EPHY.TXP: J3.1 (TD+), R26.1
- new net LED100: R31.1
- new net LED_ACT: R30.1
- new net MPU/UART_RX: J4.2 (Pin_2)
- new net MPU/UART_TX: J4.3 (Pin_3)
- new net SDMMC.CLK: J2.5 (CLK), RN1.1 (R1.1)
- new net SDMMC.CMD: J2.3 (CMD), RN1.2 (R2.1)
- new net SDMMC.D0: J2.7 (DAT0), RN2.4 (R4.1)
- new net SDMMC.D1: J2.8 (DAT1), RN2.3 (R3.1)
- new net SDMMC.D2: J2.1 (DAT2), RN1.4 (R4.1)
- new net SDMMC.D3: J2.2 (DAT3/CD), RN1.3 (R3.1)
- new net SDMMC.DET: J2.9 (DET_B)
- new net USB.DN: J1.A7 (D-), J1.B7 (D-), U5.1 (D+)
- new net USB.DP: J1.A6 (D+), J1.B6 (D+), U5.2 (D-)
Other:
- added sheet Accelerometer (accelerometer.kicad_sch)
- added sheet Flash (flash.kicad_sch)
- added sheet OV9281 (ov9281.kicad_sch)
- added sheet OV9282 (ov9281.kicad_sch)
- sheet MPU ports: added EPHY{EPHY}, FSPI{FSPI}, I2C3{I2C}, I2C4{I2C}, LED100, LED_ACT, MIPI1{MIPI}, MIPI2{MIPI}, SDMMC{MMC1}, STROBE1, STROBE2, UART_RX, UART_TX, USB{USB}, VSYNC1, VSYNC2, XSHUTDOWN1, XSHUTDOWN2; removed MMC1
- note added: "Camera Lens"
- note added: "I2C Address: 0x20"
- note added: "I2C Address: 0xC0"
- note added: "RV1103G"
