File: 4reel_ee/accelerometer.kicad_sch (KiCad schematic)
At the start: 5 parts, among them U8 LIS2HH12

Commit message: R0.1-rc1
Parts:
- C49: MPN (none) -> CL05B104KP5VPNC
- C54: MPN (none) -> GRM155R60J106ME05D
- R21, R22: MPN (none) -> RC0402FR-074K7L
Changed lines of the file:
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@@
+			)
+		)
+		(property "MPN" "RC0402FR-074K7L"
+			(at 129.54 88.9 0)
+			(hide yes)
+			(show_name no)
+			(do_not_autoplace no)
+			(effects
+				(font
+					(size 1.27 1.27)
+				)
 			)
 		)
@@
 			)
 		)
+		(property "MPN" "CL05B104KP5VPNC"
+			(at 173.99 81.28 0)
+			(hide yes)
+			(show_name no)
+			(do_not_autoplace no)
+			(effects
+				(font
+					(size 1.27 1.27)
+				)
+			)
+		)
 		(pin "1"
 		)
@@
 			)
 		)
+		(property "MPN" "GRM155R60J106ME05D"
+			(at 185.42 81.28 0)
+			(hide yes)
+			(show_name no)
+			(do_not_autoplace no)
+			(effects
+				(font
+					(size 1.27 1.27)
+				)
+			)
+		)
 		(pin "1"
 		)
@@
 			(at 140.97 88.9 0)
 			(hide yes)
+			(show_name no)
+			(do_not_autoplace no)
+			(effects
+				(font
+					(size 1.27 1.27)
+				)
+			)
+		)
+		(property "MPN" "RC0402FR-074K7L"
+			(at 140.97 88.9 0)
+			(hide yes)
