File: 4reel_ee/flash.kicad_sch (KiCad schematic)
At the start: 2 parts, among them U7 W25Q16JVSS

Commit message: Worked on the routing
Parts:
- removed U7: W25Q16JVSS, Package_SO:SOIC-8_5.3x5.3mm_P1.27mm, symbol Memory_Flash:W25Q16JVSS
- added U7: W25Q32JVZP, Package_SON:WSON-8-1EP_6x5mm_P1.27mm_EP3.4x4.3mm, symbol Memory_Flash:W25Q32JVZP
Connections:
- net +3V3: now also U7.8 (VCC)
- net FSPI.CLK: now also U7.6 (CLK)
- net FSPI.D0: now also U7.5 (DI/IO_{0})
- net FSPI.D1: now also U7.2 (DO/IO_{1})
- net FSPI.D2: now also U7.3 (~{WP}/IO_{2})
- net FSPI.D3: now also U7.7 (~{HOLD}/~{RESET}/IO_{3})
- net FSPI.~{CS}: now also U7.1 (~{CS})
- net GND: now also U7.4 (GND)
Changed lines of the file:
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@@
 	)
 	(symbol
-		(lib_id "Memory_Flash:W25Q16JVSS")
+		(lib_id "Memory_Flash:W25Q32JVZP")
 		(at 151.13 92.71 0)
 		(unit 1)
@@
 			)
 		)
-		(property "Value" "W25Q16JVSS"
+		(property "Value" "W25Q32JVZP"
 			(at 162.56 93.9799 0)
 			(show_name no)
@@
 			)
 		)
-		(property "Footprint" "Package_SO:SOIC-8_5.3x5.3mm_P1.27mm"
+		(property "Footprint" "Package_SON:WSON-8-1EP_6x5mm_P1.27mm_EP3.4x4.3mm"
 			(at 151.13 92.71 0)
 			(hide yes)
@@
 			)
 		)
-		(property "Datasheet" "https://www.winbond.com/hq/support/documentation/levelOne.jsp?__locale=en&DocNo=DA00-W25Q16JV.1"
+		(property "Datasheet" "http://www.winbond.com/resource-files/w25q32jv%20revg%2003272018%20plus.pdf"
+			(at 151.13 95.25 0)
+			(hide yes)
+			(show_name no)
+			(do_not_autoplace no)
+			(effects
+				(font
+					(size 1.27 1.27)
+				)
+			)
+		)
+		(property "Description" "32Mbit / 4MiB Serial Flash Memory, Standard/Dual/Quad SPI, 2.7-3.6V, WSON-8"
 			(at 151.13 92.71 0)
 			(hide yes)
@@
 			)
 		)
-		(property "Description" "16Mbit / 2MiB Serial Flash Memory, Standard/Dual/Quad SPI, 2.7-3.6V, SOIC-8 (208 mil)"
+		(property "MPN" "W25Q32JVZPIQ"
 			(at 151.13 92.71 0)
 			(hide yes)
@@
 			)
 		)
-		(pin "3"
+		(pin "7"
 		)
 		(pin "2"
@@
 		(pin "1"
 		)
+		(pin "5"
+		)
 		(pin "4"
+		)
+		(pin "8"
+		)
+		(pin "9"
 		)
 		(pin "6"
 		)
-		(pin "5"
-		)
-		(pin "7"
-		)
-		(pin "8"
+		(pin "3"
 		)
 		(instances

Commit message: R0.1-rc1
Parts:
- C31: MPN (none) -> CL05B104KP5VPNC
Changed lines of the file:
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@@
+			)
+		)
+		(property "MPN" "CL05B104KP5VPNC"
+			(at 154.94 74.93 0)
+			(hide yes)
+			(show_name no)
+			(do_not_autoplace no)
+			(effects
+				(font
+					(size 1.27 1.27)
+				)
 			)
 		)
