File: 4reel_ee/4reel_ee.kicad_sch (KiCad schematic)
At the start: 22 parts, among them J1 USB_C_Receptacle_USB2.0_16P, J2 Micro_SD_Card_Det2, J3 RJ45_Hanrun_HR911105A_Horizon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, J4 JST, U5 TPD2EUSB30

Commit message: Rename
Parts:
- MP1, MP2: symbol wingcam:Camera_Lens_20mm -> 4reel:Camera_Lens_20mm
Changed lines of the file:
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@@
 		)
 		(instances
-			(project "wingcam_ee"
+			(project "4reel_ee"
 				(path "/6672ba93-cf23-43d1-a630-d60a05df29bc"
 					(reference "R29")
@@
 		)
 		(instances
-			(project "wingcam_ee"
+			(project "4reel_ee"
 				(path "/6672ba93-cf23-43d1-a630-d60a05df29bc"
 					(reference "H2")
@@
 		)
 		(instances
-			(project "wingcam_ee"
+			(project "4reel_ee"
 				(path "/6672ba93-cf23-43d1-a630-d60a05df29bc"
 					(reference "#PWR093")
@@
 		)
 		(instances
-			(project "wingcam_ee"
+			(project "4reel_ee"
 				(path "/6672ba93-cf23-43d1-a630-d60a05df29bc"
 					(reference "RN1")
@@
 	)
 	(symbol
-		(lib_id "wingcam:Camera_Lens_20mm")
+		(lib_id "4reel:Camera_Lens_20mm")
 		(at 172.72 30.48 0)
 		(unit 1)
@@
 		)
 		(instances
-			(project "wingcam_ee"
+			(project "4reel_ee"
 				(path "/6672ba93-cf23-43d1-a630-d60a05df29bc"
 					(reference "MP1")
@@
 		)
 		(instances
-			(project "wingcam_ee"
+			(project "4reel_ee"
 				(path "/6672ba93-cf23-43d1-a630-d60a05df29bc"
 					(reference "#PWR088")
@@
 		)
 		(instances
-			(project "wingcam_ee"
+			(project "4reel_ee"
 				(path "/6672ba93-cf23-43d1-a630-d60a05df29bc"
 					(reference "R28")
@@
 		)
 		(instances
-			(project "wingcam_ee"
+			(project "4reel_ee"
 				(path "/6672ba93-cf23-43d1-a630-d60a05df29bc"
 					(reference "U5")
@@
 		)
 		(instances
-			(project "wingcam_ee"
+			(project "4reel_ee"
 				(path "/6672ba93-cf23-43d1-a630-d60a05df29bc"
 					(reference "RN2")
@@
 		)
 		(instances
-			(project "wingcam_ee"
+			(project "4reel_ee"
 				(path "/6672ba93-cf23-43d1-a630-d60a05df29bc"
 					(reference "R14")
@@
 		)
 		(instances
-			(project "wingcam_ee"
+			(project "4reel_ee"
 				(path "/6672ba93-cf23-43d1-a630-d60a05df29bc"
 					(reference "#PWR01")
@@
 		)
 		(instances
-			(project "wingcam_ee"
+			(project "4reel_ee"
 				(path "/6672ba93-cf23-43d1-a630-d60a05df29bc"
 					(reference "#PWR056")
@@
 		)
 		(instances
-			(project "wingcam_ee"
+			(project "4reel_ee"
 				(path "/6672ba93-cf23-43d1-a630-d60a05df29bc"
 					(reference "H4")
@@
 		)
 		(instances
-			(project "wingcam_ee"
+			(project "4reel_ee"
 				(path "/6672ba93-cf23-43d1-a630-d60a05df29bc"
 					(reference "H3")
@@
 		)
 		(instances
-			(project "wingcam_ee"
+			(project "4reel_ee"
 				(path "/6672ba93-cf23-43d1-a630-d60a05df29bc"
 					(reference "R27")
@@
 		)
 		(instances
-			(project "wingcam_ee"
+			(project "4reel_ee"
 				(path "/6672ba93-cf23-43d1-a630-d60a05df29bc"
 					(reference "R31")
@@
 		)
 		(instances
-			(project "wingcam_ee"
+			(project "4reel_ee"
 				(path "/6672ba93-cf23-43d1-a630-d60a05df29bc"
 					(reference "#PWR062")
@@
 		)
 		(instances
-			(project "wingcam_ee"
+			(project "4reel_ee"
 				(path "/6672ba93-cf23-43d1-a630-d60a05df29bc"
 					(reference "J3")
@@
 		)
 		(instances
-			(project "wingcam_ee"
+			(project "4reel_ee"
 				(path "/6672ba93-cf23-43d1-a630-d60a05df29bc"
 					(reference "#PWR091")
@@
 		)
 		(instances
-			(project "wingcam_ee"
+			(project "4reel_ee"
 				(path "/6672ba93-cf23-43d1-a630-d60a05df29bc"
 					(reference "#PWR0127")
@@
 		)
 		(instances
-			(project "wingcam_ee"
+			(project "4reel_ee"
 				(path "/6672ba93-cf23-43d1-a630-d60a05df29bc"
 					(reference "H1")
@@
 		)
 		(instances
-			(project "wingcam_ee"
+			(project "4reel_ee"
 				(path "/6672ba93-cf23-43d1-a630-d60a05df29bc"
 					(reference "#PWR089")
@@
 		)
 		(instances
-			(project "wingcam_ee"
+			(project "4reel_ee"
 				(path "/6672ba93-cf23-43d1-a630-d60a05df29bc"
 					(reference "R26")
@@
 		)
 		(instances
-			(project "wingcam_ee"
+			(project "4reel_ee"
 				(path "/6672ba93-cf23-43d1-a630-d60a05df29bc"
 					(reference "C50")
@@
 		)
 		(instances
-			(project "wingcam_ee"
+			(project "4reel_ee"
 				(path "/6672ba93-cf23-43d1-a630-d60a05df29bc"
 					(reference "#PWR071")
@@
 		)
 		(instances
-			(project "wingcam_ee"
+			(project "4reel_ee"
 				(path "/6672ba93-cf23-43d1-a630-d60a05df29bc"
 					(reference "#PWR072")
@@
 		)
 		(instances
-			(project "wingcam_ee"
+			(project "4reel_ee"
 				(path "/6672ba93-cf23-43d1-a630-d60a05df29bc"
 					(reference "#PWR0128")
@@
 		)
 		(instances
-			(project "wingcam_ee"
+			(project "4reel_ee"
 				(path "/6672ba93-cf23-43d1-a630-d60a05df29bc"
 					(reference "#PWR092")
@@
 		)
 		(instances
-			(project "wingcam_ee"
+			(project "4reel_ee"
 				(path "/6672ba93-cf23-43d1-a630-d60a05df29bc"
 					(reference "#PWR073")
@@
 		)
 		(instances
-			(project "wingcam_ee"
+			(project "4reel_ee"
 				(path "/6672ba93-cf23-43d1-a630-d60a05df29bc"
 					(reference "#PWR0100")
@@
 		)
 		(instances
-			(project "wingcam_ee"
+			(project "4reel_ee"
 				(path "/6672ba93-cf23-43d1-a630-d60a05df29bc"
 					(reference "J1")
@@
 		)
 		(instances
-			(project "wingcam_ee"
+			(project "4reel_ee"
 				(path "/6672ba93-cf23-43d1-a630-d60a05df29bc"
 					(reference "#PWR041")
@@
 		)
 		(instances
-			(project "wingcam_ee"
+			(project "4reel_ee"
 				(path "/6672ba93-cf23-43d1-a630-d60a05df29bc"
 					(reference "R15")
@@
 		)
 		(instances
-			(project "wingcam_ee"
+			(project "4reel_ee"
 				(path "/6672ba93-cf23-43d1-a630-d60a05df29bc"
 					(reference "J2")
@@
 		)
 		(instances
-			(project "wingcam_ee"
+			(project "4reel_ee"
 				(path "/6672ba93-cf23-43d1-a630-d60a05df29bc"
 					(reference "#PWR070")
@@
 		)
 		(instances
-			(project "wingcam_ee"
+			(project "4reel_ee"
 				(path "/6672ba93-cf23-43d1-a630-d60a05df29bc"
 					(reference "R30")
@@
 		)
 		(instances
-			(project "wingcam_ee"
+			(project "4reel_ee"
 				(path "/6672ba93-cf23-43d1-a630-d60a05df29bc"
 					(reference "J4")
@@
 		)
 		(instances
-			(project "wingcam_ee"
+			(project "4reel_ee"
 				(path "/6672ba93-cf23-43d1-a630-d60a05df29bc"
 					(reference "#PWR02")
@@
 	)
 	(symbol
-		(lib_id "wingcam:Camera_Lens_20mm")
+		(lib_id "4reel:Camera_Lens_20mm")
 		(at 204.47 30.48 0)
 		(unit 1)
@@
 		)
 		(instances
-			(project "wingcam_ee"
+			(project "4reel_ee"
 				(path "/6672ba93-cf23-43d1-a630-d60a05df29bc"
 					(reference "MP2")
@@
 		)
 		(instances
-			(project "wingcam_ee"
+			(project "4reel_ee"
 				(path "/6672ba93-cf23-43d1-a630-d60a05df29bc"
 					(reference "#PWR099")
@@
 		)
 		(instances
-			(project "wingcam_ee"
+			(project "4reel_ee"
 				(path "/6672ba93-cf23-43d1-a630-d60a05df29bc"
 					(reference "#PWR090")
@@
 		)
 		(instances
-			(project "wingcam_ee"
+			(project "4reel_ee"
 				(path "/6672ba93-cf23-43d1-a630-d60a05df29bc"
 					(page "2")
@@
 		)
 		(instances
-			(project "wingcam_ee"
+			(project "4reel_ee"
 				(path "/6672ba93-cf23-43d1-a630-d60a05df29bc"
 					(page "4")
@@
 		)
 		(instances
-			(project "wingcam_ee"
+			(project "4reel_ee"
 				(path "/6672ba93-cf23-43d1-a630-d60a05df29bc"
 					(page "5")
@@
 		)
 		(instances
-			(project "wingcam_ee"
+			(project "4reel_ee"
 				(path "/6672ba93-cf23-43d1-a630-d60a05df29bc"
 					(page "6")
@@
 		)
 		(instances
-			(project "wingcam_ee"
+			(project "4reel_ee"
 				(path "/6672ba93-cf23-43d1-a630-d60a05df29bc"
 					(page "7")
@@
 		)
 		(instances
-			(project "wingcam_ee"
+			(project "4reel_ee"
 				(path "/6672ba93-cf23-43d1-a630-d60a05df29bc"
 					(page "3")

Commit message: Worked on the routing
Parts:
- removed R26, R27, R28, R29: 49.9R, Resistor_SMD:R_0402_1005Metric, symbol Device:R_Small
- added C73, C74: 10nF, Capacitor_SMD:C_0402_1005Metric, symbol Device:C_Small
Connections:
- net +3V3: no longer J3.4 (TCT), J3.5 (RCT)
- net GND: now also C73.2, C74.2
- new net: C74.1, J3.5 (RCT)
- new net: C73.1, J3.4 (TCT)

Commit message: Worked on the routing.
Connections:
- net MPU/UART_RX: now also J4.3 (Pin_3); no longer J4.2 (Pin_2)
- net MPU/UART_TX: now also J4.2 (Pin_2); no longer J4.3 (Pin_3)
- no-connect marks 0 -> 1
Other:
- sheet MPU ports: added VSYNC, XSHUTDOWN; removed VSYNC1, VSYNC2, XSHUTDOWN1, XSHUTDOWN2
- sheet OV9281 ports: added DVDD; removed none
- sheet OV9282 ports: added DVDD; removed none
Changed lines of the file:
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@@
 	)
 	(junction
+		(at 227.33 113.03)
+		(diameter 0)
+		(color 0 0 0 0)
+	)
+	(junction
 		(at 96.52 130.81)
 		(diameter 0)
@@
 	)
 	(junction
+		(at 224.79 115.57)
+		(diameter 0)
+		(color 0 0 0 0)
+	)
+	(junction
 		(at 115.57 130.81)
 		(diameter 0)
@@
 		(color 0 0 0 0)
 	)
+	(no_connect
+		(at 264.16 133.35)
+	)
 	(bus_entry
 		(at 134.62 173.99)
@@
 	(wire
 		(pts
-			(xy 213.36 139.7) (xy 243.84 139.7)
+			(xy 227.33 113.03) (xy 243.84 113.03)
 		)
 		(stroke
@@
 	(wire
 		(pts
+			(xy 224.79 142.24) (xy 243.84 142.24)
+		)
+		(stroke
+			(width 0)
+			(type default)
+		)
+	)
+	(wire
+		(pts
 			(xy 39.37 100.33) (xy 39.37 101.6)
 		)
@@
 	(wire
 		(pts
+			(xy 224.79 115.57) (xy 224.79 142.24)
+		)
+		(stroke
+			(width 0)
+			(type default)
+		)
+	)
+	(wire
+		(pts
 			(xy 82.55 171.45) (xy 114.3 171.45)
 		)
@@
 	(wire
 		(pts
+			(xy 224.79 115.57) (xy 243.84 115.57)
+		)
+		(stroke
+			(width 0)
+			(type default)
+		)
+	)
+	(wire
+		(pts
 			(xy 100.33 143.51) (xy 100.33 163.83)
 		)
@@
 	(wire
 		(pts
+			(xy 243.84 139.7) (xy 227.33 139.7)
+		)
+		(stroke
+			(width 0)
+			(type default)
+		)
+	)
+	(wire
+		(pts
 			(xy 76.2 43.18) (xy 83.82 43.18)
 		)
@@
 	(wire
 		(pts
-			(xy 213.36 115.57) (xy 243.84 115.57)
+			(xy 213.36 115.57) (xy 224.79 115.57)
 		)
 		(stroke
@@
 	(wire
 		(pts
-			(xy 213.36 113.03) (xy 243.84 113.03)
+			(xy 213.36 113.03) (xy 227.33 113.03)
 		)
 		(stroke
@@
 	(wire
 		(pts
-			(xy 213.36 142.24) (xy 243.84 142.24)
+			(xy 82.55 156.21) (xy 95.25 156.21)
 		)
 		(stroke
@@
 	(wire
 		(pts
-			(xy 82.55 156.21) (xy 95.25 156.21)
+			(xy 158.75 78.74) (xy 170.18 78.74)
 		)
 		(stroke
@@
 	(wire
 		(pts
-			(xy 158.75 78.74) (xy 170.18 78.74)
+			(xy 97.79 130.81) (xy 100.33 130.81)
 		)
 		(stroke
@@
 	(wire
 		(pts
-			(xy 97.79 130.81) (xy 100.33 130.81)
+			(xy 96.52 130.81) (xy 97.79 130.81)
 		)
 		(stroke
@@
 	(wire
 		(pts
-			(xy 96.52 130.81) (xy 97.79 130.81)
+			(xy 114.3 130.81) (xy 115.57 130.81)
 		)
 		(stroke
@@
 	(wire
 		(pts
-			(xy 114.3 130.81) (xy 115.57 130.81)
+			(xy 82.55 158.75) (xy 97.79 158.75)
 		)
 		(stroke
@@
 	(wire
 		(pts
-			(xy 82.55 158.75) (xy 97.79 158.75)
+			(xy 95.25 130.81) (xy 96.52 130.81)
 		)
 		(stroke
@@
 	(wire
 		(pts
-			(xy 95.25 130.81) (xy 96.52 130.81)
+			(xy 264.16 107.95) (xy 266.7 107.95)
 		)
 		(stroke
@@
 	(wire
 		(pts
+			(xy 227.33 139.7) (xy 227.33 113.03)
+		)
+		(stroke
+			(width 0)
+			(type default)
+		)
+	)
+	(wire
+		(pts
 			(xy 266.7 110.49) (xy 266.7 107.95)
 		)
@@
 	)
 	(symbol
-		(lib_id "power:+5V")
-		(at 266.7 107.95 0)
-		(unit 1)
-		(body_style 1)
-		(exclude_from_sim no)
-		(in_bom yes)
-		(on_board yes)
-		(in_pos_files yes)
-		(dnp no)
-		(property "Reference" "#PWR0127"
-			(at 266.7 111.76 0)
-			(hide yes)
-			(show_name no)
-			(do_not_autoplace no)
-			(effects
-				(font
-					(size 1.27 1.27)
-				)
-			)
-		)
-		(property "Value" "+1V8"
-			(at 268.732 104.14 0)
-			(show_name no)
-			(do_not_autoplace no)
-			(effects
-				(font
-					(size 1.27 1.27)
-				)
-			)
-		)
-		(property "Footprint" ""
-			(at 266.7 107.95 0)
-			(hide yes)
-			(show_name no)
-			(do_not_autoplace no)
-			(effects
-				(font
-					(size 1.27 1.27)
-				)
-			)
-		)
-		(property "Datasheet" ""
-			(at 266.7 107.95 0)
-			(hide yes)
-			(show_name no)
-			(do_not_autoplace no)
-			(effects
-				(font
-					(size 1.27 1.27)
-				)
-			)
-		)
-		(property "Description" "Power symbol creates a global label with name \"+5V\""
-			(at 266.7 107.95 0)
-			(hide yes)
-			(show_name no)
-			(do_not_autoplace no)
-			(effects
-				(font
-					(size 1.27 1.27)
-				)
-			)
-		)
-		(pin "1"
-		)
-		(instances
-			(project "4reel_ee"
-				(path "/6672ba93-cf23-43d1-a630-d60a05df29bc"
-					(reference "#PWR0127")
-					(unit 1)
-				)
-			)
-		)
-	)
-	(symbol
 		(lib_id "Mechanical:MountingHole")
 		(at 176.53 44.45 0)
@@
 			)
 		)
-		(pin "VSYNC1" bidirectional
+		(pin "VSYNC" bidirectional
 			(at 213.36 113.03 0)
 			(effects
@@
 			)
 		)
-		(pin "XSHUTDOWN1" bidirectional
+		(pin "XSHUTDOWN" bidirectional
 			(at 213.36 115.57 0)
 			(effects
@@
 		)
 		(pin "UART_RX" bidirectional
-			(at 170.18 76.2 180)
+			(at 170.18 78.74 180)
 			(effects
 				(font
@@
 		)
 		(pin "UART_TX" bidirectional
-			(at 170.18 78.74 180)
+			(at 170.18 76.2 180)
 			(effects
 				(font
@@
 			)
 		)
-		(pin "VSYNC2" bidirectional
-			(at 213.36 139.7 0)
-			(effects
-				(font
-					(size 1.27 1.27)
-				)
-				(justify right)
-			)
-		)
-		(pin "XSHUTDOWN2" bidirectional
-			(at 213.36 142.24 0)
-			(effects
-				(font
-					(size 1.27 1.27)
-				)
-				(justify right)
-			)
-		)
 		(instances
 			(project "4reel_ee"
@@
 			)
 		)
+		(pin "DVDD" bidirectional
+			(at 264.16 107.95 0)
+			(effects
+				(font
+					(size 1.27 1.27)
+				)
+				(justify right)
+			)
+		)
 		(instances
 			(project "4reel_ee"
@@
 			(effects
 				(font
+					(size 1.27 1.27)
+				)
+				(justify right)
+			)
+		)
+		(pin "DVDD" bidirectional
+			(at 264.16 133.35 0)
+			(effects
+				(font

Commit message: Finished initial rough layout.
Parts:
- added FID1, FID2, FID3, FID4, FID5, FID6: Fiducial, Fiducial:Fiducial_0.5mm_Mask1.5mm, symbol Mechanical:Fiducial

Commit message: R0.1-rc1
Parts:
- C50: MPN (none) -> GRM155R60J106ME05D
- C73, C74: MPN (none) -> C0402C103K5REC7411
- J3: MPN (none) -> HR911105A
- J4: MPN (none) -> SM04B-SRSS-TB
- R14, R15: MPN (none) -> RC0402FR-075K6L
- R30, R31: MPN (none) -> RC0402FR-07330RL
- U5: MPN (none) -> TPD2EUSB30ADRTR
Connections:
- net GND: now also J2.10 (DET_A)
- net SDMMC.CLK: no longer RN1.1 (R1.1)
- net SDMMC.DET: now also RN2.1 (R1.1)
- net at RN2.2 (R2.1): no longer J2.10 (DET_A)
Changed lines of the file:
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@@
 	)
 	(junction
-		(at 100.33 163.83)
-		(diameter 0)
-		(color 0 0 0 0)
-	)
-	(junction
 		(at 227.33 113.03)
 		(diameter 0)
@@
 	)
 	(junction
+		(at 119.38 176.53)
+		(diameter 0)
+		(color 0 0 0 0)
+	)
+	(junction
 		(at 76.2 40.64)
 		(diameter 0)
@@
 	)
 	(junction
-		(at 224.79 115.57)
+		(at 97.79 130.81)
 		(diameter 0)
 		(color 0 0 0 0)
 	)
 	(junction
-		(at 115.57 130.81)
+		(at 224.79 115.57)
 		(diameter 0)
 		(color 0 0 0 0)
 	)
 	(junction
-		(at 97.79 130.81)
+		(at 115.57 130.81)
 		(diameter 0)
 		(color 0 0 0 0)
@@
 	(wire
 		(pts
-			(xy 82.55 163.83) (xy 100.33 163.83)
-		)
-		(stroke
-			(width 0)
-			(type default)
-		)
-	)
-	(wire
-		(pts
 			(xy 95.25 130.81) (xy 95.25 133.35)
 		)
@@
 	(wire
 		(pts
+			(xy 119.38 176.53) (xy 132.08 176.53)
+		)
+		(stroke
+			(width 0)
+			(type default)
+		)
+	)
+	(wire
+		(pts
+			(xy 119.38 143.51) (xy 119.38 176.53)
+		)
+		(stroke
+			(width 0)
+			(type default)
+		)
+	)
+	(wire
+		(pts
 			(xy 86.36 55.88) (xy 83.82 53.34)
 		)
@@
 	(wire
 		(pts
-			(xy 82.55 176.53) (xy 132.08 176.53)
+			(xy 82.55 176.53) (xy 119.38 176.53)
 		)
 		(stroke
@@
 	(wire
 		(pts
-			(xy 100.33 163.83) (xy 132.08 163.83)
+			(xy 82.55 163.83) (xy 132.08 163.83)
 		)
 		(stroke
@@
 	(wire
 		(pts
-			(xy 100.33 143.51) (xy 100.33 163.83)
-		)
-		(stroke
-			(width 0)
-			(type default)
-		)
-	)
-	(wire
-		(pts
 			(xy 82.55 153.67) (xy 92.71 153.67)
 		)
@@
 	(wire
 		(pts
-			(xy 110.49 40.64) (xy 116.84 40.64)
+			(xy 82.55 173.99) (xy 86.36 173.99)
 		)
 		(stroke
@@
 	(wire
 		(pts
-			(xy 116.84 173.99) (xy 116.84 143.51)
+			(xy 110.49 40.64) (xy 116.84 40.64)
 		)
 		(stroke
@@
 	(wire
 		(pts
+			(xy 100.33 130.81) (xy 100.33 133.35)
+		)
+		(stroke
+			(width 0)
+			(type default)
+		)
+	)
+	(wire
+		(pts
 			(xy 95.25 156.21) (xy 132.08 156.21)
 		)
@@
 	(wire
 		(pts
-			(xy 100.33 130.81) (xy 100.33 133.35)
+			(xy 83.82 104.14) (xy 138.43 104.14)
 		)
 		(stroke
@@
 	(wire
 		(pts
-			(xy 83.82 104.14) (xy 138.43 104.14)
+			(xy 97.79 130.81) (xy 100.33 130.81)
 		)
 		(stroke
@@
 	(wire
 		(pts
-			(xy 97.79 130.81) (xy 100.33 130.81)
-		)
-		(stroke
-			(width 0)
-			(type default)
-		)
-	)
-	(wire
-		(pts
 			(xy 96.52 130.81) (xy 97.79 130.81)
 		)
@@
 	(wire
 		(pts
-			(xy 82.55 173.99) (xy 116.84 173.99)
-		)
-		(stroke
-			(width 0)
-			(type default)
-		)
-	)
-	(wire
-		(pts
 			(xy 40.64 104.14) (xy 31.75 104.14)
 		)
@@
 			)
 		)
+		(property "MPN" "TPD2EUSB30ADRTR"
+			(at 96.52 55.88 0)
+			(hide yes)
+			(show_name no)
+			(do_not_autoplace no)
+			(effects
+				(font
+					(size 1.27 1.27)
+				)
+			)
+		)
 		(pin "1"
 		)
@@
 			)
 		)
+		(property "MPN" "C0402C103K5REC7411"
+			(at 91.44 101.6 90)
+			(hide yes)
+			(show_name no)
+			(do_not_autoplace no)
+			(effects
+				(font
+					(size 1.27 1.27)
+				)
+			)
+		)
 		(pin "1"
 		)
@@
 			)
 		)
+		(property "MPN" "RC0402FR-075K6L"
+			(at 80.01 30.48 90)
+			(hide yes)
+			(show_name no)
+			(do_not_autoplace no)
+			(effects
+				(font
+					(size 1.27 1.27)
+				)
+			)
+		)
 		(pin "1"
 		)
@@
 			)
 		)
+		(property "MPN" "RC0402FR-07330RL"
+			(at 29.21 104.14 90)
+			(hide yes)
+			(show_name no)
+			(do_not_autoplace no)
+			(effects
+				(font
+					(size 1.27 1.27)
+				)
+			)
+		)
 		(pin "1"
 		)
@@
 			)
 		)
+		(property "MPN" "HR911105A"
+			(at 63.5 99.06 0)
+			(hide yes)
+			(show_name no)
+			(do_not_autoplace no)
+			(effects
+				(font
+					(size 1.27 1.27)
+				)
+			)
+		)
 		(pin "11"
 		)
@@
 			)
 		)
+		(property "MPN" "GRM155R60J106ME05D"
+			(at 34.29 161.29 0)
+			(hide yes)
+			(show_name no)
+			(do_not_autoplace no)
+			(effects
+				(font
+					(size 1.27 1.27)
+				)
+			)
+		)
 		(pin "1"
 		)
@@
 	(symbol
 		(lib_id "power:GND")
+		(at 86.36 173.99 90)
+		(unit 1)
+		(body_style 1)
+		(exclude_from_sim no)
+		(in_bom yes)
+		(on_board yes)
+		(in_pos_files yes)
+		(dnp no)
+		(fields_autoplaced yes)
+		(property "Reference" "#PWR0123"
+			(at 92.71 173.99 0)
+			(hide yes)
+			(show_name no)
+			(do_not_autoplace no)
+			(effects
+				(font
+					(size 1.27 1.27)
+				)
+			)
+		)
+		(property "Value" "GND"
+			(at 91.44 173.99 0)
+			(hide yes)
+			(show_name no)
+			(do_not_autoplace no)
+			(effects
+				(font
+					(size 1.27 1.27)
+				)
+			)
+		)
+		(property "Footprint" ""
+			(at 86.36 173.99 0)
+			(hide yes)
+			(show_name no)
+			(do_not_autoplace no)
+			(effects
+				(font
+					(size 1.27 1.27)
+				)
+			)
+		)
+		(property "Datasheet" ""
+			(at 86.36 173.99 0)
+			(hide yes)
+			(show_name no)
+			(do_not_autoplace no)
+			(effects
+				(font
+					(size 1.27 1.27)
+				)
+			)
+		)
+		(property "Description" "Power symbol creates a global label with name \"GND\" , ground"
+			(at 86.36 173.99 0)
+			(hide yes)
+			(show_name no)
+			(do_not_autoplace no)
+			(effects
+				(font
+					(size 1.27 1.27)
+				)
+			)
+		)
+		(pin "1"
+		)
+		(instances
+			(project "4reel_ee"
+				(path "/6672ba93-cf23-43d1-a630-d60a05df29bc"
+					(reference "#PWR0123")
+					(unit 1)
+				)
+			)
+		)
+	)
+	(symbol
+		(lib_id "power:GND")
 		(at 86.36 35.56 0)
 		(unit 1)
@@
 			)
 		)
+		(property "MPN" "RC0402FR-075K6L"
+			(at 80.01 33.02 90)
+			(hide yes)
+			(show_name no)
+			(do_not_autoplace no)
+			(effects
+				(font
+					(size 1.27 1.27)
+				)
+			)
+		)
 		(pin "1"
 		)
@@
 			)
 		)
+		(property "MPN" "RC0402FR-07330RL"
+			(at 29.21 93.98 90)
+			(hide yes)
+			(show_name no)
+			(do_not_autoplace no)
+			(effects
+				(font
+					(size 1.27 1.27)
+				)
+			)
+		)
 		(pin "1"
 		)
@@
 			)
 		)
+		(property "MPN" "SM04B-SRSS-TB"
+			(at 153.67 76.2 0)
+			(hide yes)
+			(show_name no)
+			(do_not_autoplace no)
+			(effects
+				(font
+					(size 1.27 1.27)
+				)
+			)
+		)
 		(pin "2"
 		)
@@
 			(hide yes)
 			(show_name no)
+			(do_not_autoplace no)
+			(effects
+				(font
+					(size 1.27 1.27)
+				)
+			)
+		)
+		(property "MPN" "C0402C103K5REC7411"
+			(at 91.44 93.98 90)
+			(hide yes)
+			(show_name no)

Commit message: R0.1 release.
Other:
- sheet OV9281 ports: added DOVDD; removed DVDD
- sheet OV9282 ports: added DOVDD; removed DVDD
Changed lines of the file:
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@@
 			)
 		)
-		(pin "DVDD" bidirectional
+		(pin "DOVDD" bidirectional
 			(at 264.16 107.95 0)
 			(effects
@@
 			)
 		)
-		(pin "DVDD" bidirectional
+		(pin "DOVDD" bidirectional
 			(at 264.16 133.35 0)
 			(effects

Commit message: Correctd RV1103B part.
Other:
- note added: "RV1103B"
- note removed: "RV1103G"
Changed lines of the file:
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@@
 		)
 	)
-	(text "RV1103G"
+	(text "RV1103B"
 		(exclude_from_sim no)
 		(at 192.024 72.136 0)
