File: 4reel_ee/mpu.kicad_sch (KiCad schematic)
At the start: 31 parts, among them U1 RV1103G, Y2 24Mhz

Commit message: Rename
Parts:
- U1: symbol wingcam:RV1103G -> 4reel:RV1103G

Commit message: Worked on the routing
Parts:
- added C75: 100nF, Capacitor_SMD:C_0402_1005Metric, symbol Device:C_Small
Connections:
- net +0V9: now also C75.1
- net GND: now also C75.2
- net STROBE1: no longer U1.60 (PWM9_M1)
- net STROBE2: now also U1.60 (PWM9_M1)
- net VSYNC1: no longer U1.61 (PWM8_M1)
- net VSYNC2: now also U1.61 (PWM8_M1)
- net XSHUTDOWN1: no longer U1.64 (PWM4_M2)
- net XSHUTDOWN2: now also U1.64 (PWM4_M2)
Other:
- moved on the sheet: C17, C18, C19, C20

Commit message: Worked on the routing.
Connections:
- net LED100: now also U1.52 (PWM10_M1)
- net LED_ACT: now also U1.57 (PWM3_IR_M2)
- net STROBE1: now also U1.65 (PWM2_M2)
- net VSYNC2 renamed VSYNC
- net XSHUTDOWN2 renamed XSHUTDOWN
Changed lines of the file:
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@@
+	(wire
+		(pts
+			(xy 43.18 57.15) (xy 52.07 57.15)
+		)
+		(stroke
+			(width 0)
+			(type default)
+		)
+	)
 	(wire
 		(pts
@@
 		(pts
 			(xy 185.42 132.08) (xy 185.42 129.54)
+		)
+		(stroke
+			(width 0)
+			(type default)
+		)
+	)
+	(wire
+		(pts
+			(xy 43.18 59.69) (xy 52.07 59.69)
+		)
+		(stroke
+			(width 0)
+			(type default)
+		)
+	)
+	(wire
+		(pts
+			(xy 43.18 74.93) (xy 52.07 74.93)
 		)
 		(stroke
@@
 		)
 	)
-	(hierarchical_label "VSYNC2"
+	(hierarchical_label "VSYNC"
 		(shape bidirectional)
 		(at 43.18 69.85 180)
@@
 		)
 	)
-	(hierarchical_label "XSHUTDOWN1"
-		(shape bidirectional)
-		(at 68.58 121.92 180)
-		(effects
-			(font
-				(size 1.27 1.27)
-			)
-			(justify right)
-		)
-	)
 	(hierarchical_label "STROBE2"
 		(shape bidirectional)
@@
 	(hierarchical_label "LED_ACT"
 		(shape bidirectional)
-		(at 57.15 111.76 0)
-		(effects
-			(font
-				(size 1.27 1.27)
-			)
-			(justify left)
+		(at 43.18 59.69 180)
+		(effects
+			(font
+				(size 1.27 1.27)
+			)
+			(justify right)
 		)
 	)
 	(hierarchical_label "LED100"
 		(shape bidirectional)
-		(at 57.15 114.3 0)
-		(effects
-			(font
-				(size 1.27 1.27)
-			)
-			(justify left)
+		(at 43.18 74.93 180)
+		(effects
+			(font
+				(size 1.27 1.27)
+			)
+			(justify right)
 		)
 	)
@@
 	(hierarchical_label "STROBE1"
 		(shape bidirectional)
-		(at 68.58 127 180)
+		(at 43.18 57.15 180)
 		(effects
 			(font
@@
 		)
 	)
-	(hierarchical_label "XSHUTDOWN2"
+	(hierarchical_label "XSHUTDOWN"
 		(shape bidirectional)
 		(at 43.18 62.23 180)
 		(effects
 			(font
-				(size 1.27 1.27)
-			)
-			(justify right)
-		)
-	)
-	(hierarchical_label "VSYNC1"
-		(shape bidirectional)
-		(at 68.58 124.46 180)
-		(effects
-			(font

Commit message: R0.1-rc1
Parts:
- added R26: 10k, Resistor_SMD:R_0402_1005Metric, symbol Device:R_Small
- added R27: 22R, Resistor_SMD:R_0201_0603Metric, symbol Device:R_Small
- C17, C19, C20, C21, C22, C23, C25, C26, C27: MPN (none) -> GRM155R60J106ME05D
- C18, C24, C28, C75: MPN (none) -> CL05B104KP5VPNC
- C32, C38: MPN (none) -> GCM1555C1H100JA16D
- D1, D2: MPN (none) -> LTST-C281KGKT
- R10: MPN (none) -> RC0402FR-07240RL
- R11, R12: MPN (none) -> RC0402FR-074K7L
- R16, R19: MPN (none) -> RC0402FR-0722RL
- R17, R18: MPN (none) -> RC0402FR-0710KL
- R20: MPN (none) -> RC0402FR-071ML
- R23, R24: MPN (none) -> RC0402FR-071KL
- R25: MPN (none) -> RC0402FR-076K04L
- U1: MPN (none) -> RV1103G
Connections:
- net +1V8: now also R26.2
- net SDMMC.CLK: now also R27.2; no longer U1.11 (SDMMC_CLK)
- net at U1.16 (SARADC_IN0): now also R26.1
- new net: R27.1, U1.11 (SDMMC_CLK)

Commit message: R0.1 release.
Parts:
- added TP3, TP4, TP5, TP6: TestPoint, TestPoint:TestPoint_Pad_1.0x1.0mm, symbol Connector:TestPoint
- U1: MPN RV1103G -> RV1103BG3
Connections:
- net I2C3.SCL: now also TP5.1
- net I2C3.SDA: now also TP6.1
- net I2C4.SCL: now also TP3.1
- net I2C4.SDA: now also TP4.1

Commit message: Initial schematic, routing finished for RV1106 based design.
Parts:
- removed R16: 22R, Resistor_SMD:R_0402_1005Metric, symbol Device:R_Small
- removed R17, R18, R26: 10k, Resistor_SMD:R_0402_1005Metric, symbol Device:R_Small
- removed R25: 6.04k, Resistor_SMD:R_0402_1005Metric, symbol Device:R_Small
- removed U1: RV1103G, rv1103b:Rockchip_QFN-88-1EP_9x9mm_P0.35mm_EP6.5x6.5mm, symbol 4reel:RV1103G
- added C76, C78, C80, C86, C87, C88, C89, C90, C91: 100nF, Capacitor_SMD:C_0201_0603Metric, symbol Device:C_Small
- added C77: 10uF, Capacitor_SMD:C_0402_1005Metric, symbol Device:C_Small
- added R28: 22R, Resistor_SMD:R_0201_0603Metric, symbol Device:R_Small
- added U1: RV1106G3, rv1106:Rockchip_QFN-128-1EP_12.3x12.3mm_P0.35mm_EP7x7mm, symbol 4reel:RV1106G3
- C18, C24, C28, C75: footprint Capacitor_SMD:C_0402_1005Metric -> Capacitor_SMD:C_0201_0603Metric; MPN CL05B104KP5VPNC -> (none)
- R10: footprint Resistor_SMD:R_0402_1005Metric -> Resistor_SMD:R_0201_0603Metric; MPN RC0402FR-07240RL -> (none)
Connections:
- net +0V9: now also C87.1, C89.1, U1.10 (DVDD_1), U1.103 (DVDD_6), U1.115 (CPU_DVDD), U1.116 (DVDD_7), U1.51 (DVDD_2), U1.54 (DVDD_3), U1.55 (DVDD_4), U1.67 (PMU_DVDD0V9), U1.71 (OSC_PLL_DVDD), U1.82 (DVDD_5)
- net +1V8: now also C78.1, C86.1, U1.1 (MIPI_AVDD1V8), U1.24 (SARADC_USB_AVDD1V8), U1.31 (CODEC_AVDD1V8), U1.53 (DDR_PLL_AVDD1V8), U1.70 (OSC_AVDD1V8), U1.88 (GPIO6_VCC), U1.96 (OTP_AVDD1V8)
- net +3V3: now also C80.1, C88.1, C90.1, C91.1, U1.101 (ETH_AVDD3V3), U1.108 (GPIO5_VCC), U1.13 (GPIO4_VCC), U1.19 (RTC_AVDD3V3), U1.28 (USB_AVDD3V3), U1.43 (GPIO3_VCC), U1.61 (PMU_VCC3V3), U1.81 (GPIO1_VCC3V3)
- net GND: now also C76.2, C77.2, C78.2, C80.2, C86.2, C87.2, C88.2, C89.2, C90.2, C91.2, U1.129 (VSS), U1.37 (CODEC_AVSS), U1.57 (TVSS)
- net I2C3.SCL: now also U1.107 (UART0_RTS_M1)
- net I2C3.SDA: now also U1.106 (UART0_CTS_M1)
- net I2C4.SCL: now also U1.93 (VO_LCDC_D5)
- net I2C4.SDA: now also U1.92 (VO_LCDC_D4)
- net LED1: now also U1.4 (MIPI_CLK1_OUT)
- net LED2: now also U1.3 (VI_CIF_VSYNC_M0)
- net MIPI1.CK0N: now also U1.125 (MIPI_CSI_RX_CK0N)
- net MIPI1.CK0P: now also U1.126 (MIPI_CSI_RX_CK0P)
- net MIPI1.D0N: now also U1.127 (MIPI_CSI_RX_D0N)
- net MIPI1.D0P: now also U1.128 (MIPI_CSI_RX_D0P)
- net MIPI1.D1N: now also U1.123 (MIPI_CSI_RX_D1N)
- net MIPI1.D1P: now also U1.124 (MIPI_CSI_RX_D1P)
- net MIPI2.CK0N: now also U1.119 (MIPI_CSI_RX_CK1N)
- net MIPI2.CK0P: now also U1.120 (MIPI_CSI_RX_CK1P)
- net MIPI2.D0N: now also U1.121 (MIPI_CSI_RX_D2N)
- net MIPI2.D0P: now also U1.122 (MIPI_CSI_RX_D2P)
- net MIPI2.D1N: now also U1.117 (MIPI_CSI_RX_D3N)
- net MIPI2.D1P: now also U1.118 (MIPI_CSI_RX_D3P)
- net STROBE1: now also U1.83 (VO_LCDC_D1)
- net STROBE2: now also U1.84 (VO_LCDC_D0)
- net UART_RX: now also U1.105 (UART0_RX_M1)
- net UART_TX: now also U1.104 (UART0_TX_M1)
- net USB.DN: now also U1.26 (USB_DM)
- net USB.DP: now also U1.27 (USB_DP)
- net VSYNC: now also U1.86 (VO_LCDC_VSYNC)
- net XSHUTDOWN: now also U1.87 (VO_LCDC_HSYNC)
- net at C32.1, R20.2, Y2.1: now also U1.69 (OSC_XOUT)
- net at R10.2: now also U1.52 (DRAM_ZQ)
- net at R19.2, R20.1: now also U1.68 (OSC_XIN)
- net at R27.1: now also U1.15 (SDMMC0_CLK)
- net SDMMC.CLK renamed SDMMC1.CLK
- new net: R28.1, U1.111 (SDMMC1_CLK_M0)
- new net +1V35: C76.1, C77.1, U1.49 (DDR_VDDQ_1), U1.50 (DDR_VDDQ_2), U1.56 (DDR_VDDQ_3)
- new net BT_HOST_WAKE: U1.44 (FSPI_D2)
- new net BT_LPO: U1.39 (FSPI_D3)
- new net BT_RST_N: U1.48 (FSPI_CLK)
- new net BT_WAKE: U1.47 (FSPI_CS0)
- new net SDMMC1.CMD: U1.16 (SDMMC0_CMD)
- new net SDMMC1.D0: U1.14 (SDMMC0_D0)
- new net SDMMC1.D1: U1.12 (SDMMC0_D1)
- new net SDMMC1.D2: U1.18 (SDMMC0_D2)
- new net SDMMC1.D3: U1.17 (SDMMC0_D3)
- new net SDMMC1.DET: U1.11 (SDMMC0_DET)
- new net SDMMC2.CLK: R28.2
- new net SDMMC2.CMD: U1.112 (SDMMC1_CMD_M0)
- new net SDMMC2.D0: U1.110 (SDMMC1_D0_M0)
- new net SDMMC2.D1: U1.109 (SDMMC1_D1_M0)
- new net SDMMC2.D2: U1.114 (SDMMC1_D2_M0)
- new net SDMMC2.D3: U1.113 (SDMMC1_D3_M0)
- new net UART1.RXD: U1.76 (UART1_RX_M0)
- new net UART1.TXD: U1.75 (UART1_TX_M0)
- new net UART1.~{CTS}: U1.65 (I2C1_SDA_M0)
- new net UART1.~{RTS}: U1.64 (I2C1_SCL_M0)
- new net WL_HOST_WAKE: U1.41 (FSPI_D0)
- new net WL_REG_ON: U1.42 (FSPI_D1)
- no-connect marks 5 -> 40
Other:
- note added: "1.8V Logic Levels GPIO6_VCC"
- note removed: "Pins 62/63 I2C4_M1 -> VCCIO6_VCC domain -> 1.8V Pins 54/55 I2C3_M1 -> VCCIO1_VCC3V3 domain Pins 4/5 I2C4_M2 -> GPIO3_VCC domain"
- moved on the sheet: C17, C18, C19, C20, C21, C22, C23, C24, C25, C26, C27, C28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
