File: 4reel_ee/ov9281.kicad_sch (KiCad schematic)
At the start: 23 parts, among them U3 ImageSensor_OV9281, Y1 TXC-7C

Commit message: Rename
Parts:
- U3: symbol wingcam:OV9281 -> 4reel:OV9281
Changed lines of the file:
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@@
 		)
 		(instances
-			(project "wingcam_ee"
+			(project "4reel_ee"
 				(path "/6672ba93-cf23-43d1-a630-d60a05df29bc/45ac4961-8d3d-4c84-aa6c-b96cc3397d34"
 					(reference "#PWR063")
@@
 		)
 		(instances
-			(project "wingcam_ee"
+			(project "4reel_ee"
 				(path "/6672ba93-cf23-43d1-a630-d60a05df29bc/45ac4961-8d3d-4c84-aa6c-b96cc3397d34"
 					(reference "#PWR068")
@@
 		)
 		(instances
-			(project "wingcam_ee"
+			(project "4reel_ee"
 				(path "/6672ba93-cf23-43d1-a630-d60a05df29bc/45ac4961-8d3d-4c84-aa6c-b96cc3397d34"
 					(reference "#PWR057")
@@
 		)
 		(instances
-			(project "wingcam_ee"
+			(project "4reel_ee"
 				(path "/6672ba93-cf23-43d1-a630-d60a05df29bc/45ac4961-8d3d-4c84-aa6c-b96cc3397d34"
 					(reference "C40")
@@
 		)
 		(instances
-			(project "wingcam_ee"
+			(project "4reel_ee"
 				(path "/6672ba93-cf23-43d1-a630-d60a05df29bc/45ac4961-8d3d-4c84-aa6c-b96cc3397d34"
 					(reference "#PWR061")
@@
 		)
 		(instances
-			(project "wingcam_ee"
+			(project "4reel_ee"
 				(path "/6672ba93-cf23-43d1-a630-d60a05df29bc/45ac4961-8d3d-4c84-aa6c-b96cc3397d34"
 					(reference "C43")
@@
 		)
 		(instances
-			(project "wingcam_ee"
+			(project "4reel_ee"
 				(path "/6672ba93-cf23-43d1-a630-d60a05df29bc/45ac4961-8d3d-4c84-aa6c-b96cc3397d34"
 					(reference "L5")
@@
 		)
 		(instances
-			(project "wingcam_ee"
+			(project "4reel_ee"
 				(path "/6672ba93-cf23-43d1-a630-d60a05df29bc/45ac4961-8d3d-4c84-aa6c-b96cc3397d34"
 					(reference "C46")
@@
 		)
 		(instances
-			(project "wingcam_ee"
+			(project "4reel_ee"
 				(path "/6672ba93-cf23-43d1-a630-d60a05df29bc/45ac4961-8d3d-4c84-aa6c-b96cc3397d34"
 					(reference "Y1")
@@
 		)
 		(instances
-			(project "wingcam_ee"
+			(project "4reel_ee"
 				(path "/6672ba93-cf23-43d1-a630-d60a05df29bc/45ac4961-8d3d-4c84-aa6c-b96cc3397d34"
 					(reference "#PWR069")
@@
 		)
 		(instances
-			(project "wingcam_ee"
+			(project "4reel_ee"
 				(path "/6672ba93-cf23-43d1-a630-d60a05df29bc/45ac4961-8d3d-4c84-aa6c-b96cc3397d34"
 					(reference "#PWR065")
@@
 		)
 		(instances
-			(project "wingcam_ee"
+			(project "4reel_ee"
 				(path "/6672ba93-cf23-43d1-a630-d60a05df29bc/45ac4961-8d3d-4c84-aa6c-b96cc3397d34"
 					(reference "C47")
@@
 		)
 		(instances
-			(project "wingcam_ee"
+			(project "4reel_ee"
 				(path "/6672ba93-cf23-43d1-a630-d60a05df29bc/45ac4961-8d3d-4c84-aa6c-b96cc3397d34"
 					(reference "#PWR098")
@@
 		)
 		(instances
-			(project "wingcam_ee"
+			(project "4reel_ee"
 				(path "/6672ba93-cf23-43d1-a630-d60a05df29bc/45ac4961-8d3d-4c84-aa6c-b96cc3397d34"
 					(reference "#PWR048")
@@
 		)
 		(instances
-			(project "wingcam_ee"
+			(project "4reel_ee"
 				(path "/6672ba93-cf23-43d1-a630-d60a05df29bc/45ac4961-8d3d-4c84-aa6c-b96cc3397d34"
 					(reference "#PWR067")
@@
 		)
 		(instances
-			(project "wingcam_ee"
+			(project "4reel_ee"
 				(path "/6672ba93-cf23-43d1-a630-d60a05df29bc/45ac4961-8d3d-4c84-aa6c-b96cc3397d34"
 					(reference "C53")
@@
 		)
 		(instances
-			(project "wingcam_ee"
+			(project "4reel_ee"
 				(path "/6672ba93-cf23-43d1-a630-d60a05df29bc/45ac4961-8d3d-4c84-aa6c-b96cc3397d34"
 					(reference "#PWR053")
@@
 		)
 		(instances
-			(project "wingcam_ee"
+			(project "4reel_ee"
 				(path "/6672ba93-cf23-43d1-a630-d60a05df29bc/45ac4961-8d3d-4c84-aa6c-b96cc3397d34"
 					(reference "C44")
@@
 		)
 		(instances
-			(project "wingcam_ee"
+			(project "4reel_ee"
 				(path "/6672ba93-cf23-43d1-a630-d60a05df29bc/45ac4961-8d3d-4c84-aa6c-b96cc3397d34"
 					(reference "C42")
@@
 		)
 		(instances
-			(project "wingcam_ee"
+			(project "4reel_ee"
 				(path "/6672ba93-cf23-43d1-a630-d60a05df29bc/45ac4961-8d3d-4c84-aa6c-b96cc3397d34"
 					(reference "C35")
@@
 		)
 		(instances
-			(project "wingcam_ee"
+			(project "4reel_ee"
 				(path "/6672ba93-cf23-43d1-a630-d60a05df29bc/45ac4961-8d3d-4c84-aa6c-b96cc3397d34"
 					(reference "C45")
@@
 		)
 		(instances
-			(project "wingcam_ee"
+			(project "4reel_ee"
 				(path "/6672ba93-cf23-43d1-a630-d60a05df29bc/45ac4961-8d3d-4c84-aa6c-b96cc3397d34"
 					(reference "C48")
@@
 		)
 		(instances
-			(project "wingcam_ee"
+			(project "4reel_ee"
 				(path "/6672ba93-cf23-43d1-a630-d60a05df29bc/45ac4961-8d3d-4c84-aa6c-b96cc3397d34"
 					(reference "#PWR058")
@@
 		)
 		(instances
-			(project "wingcam_ee"
+			(project "4reel_ee"
 				(path "/6672ba93-cf23-43d1-a630-d60a05df29bc/45ac4961-8d3d-4c84-aa6c-b96cc3397d34"
 					(reference "#PWR064")
@@
 		)
 		(instances
-			(project "wingcam_ee"
+			(project "4reel_ee"
 				(path "/6672ba93-cf23-43d1-a630-d60a05df29bc/45ac4961-8d3d-4c84-aa6c-b96cc3397d34"
 					(reference "#PWR066")
@@
 		)
 		(instances
-			(project "wingcam_ee"
+			(project "4reel_ee"
 				(path "/6672ba93-cf23-43d1-a630-d60a05df29bc/45ac4961-8d3d-4c84-aa6c-b96cc3397d34"
 					(reference "C36")
@@
 		)
 		(instances
-			(project "wingcam_ee"
+			(project "4reel_ee"
 				(path "/6672ba93-cf23-43d1-a630-d60a05df29bc/45ac4961-8d3d-4c84-aa6c-b96cc3397d34"
 					(reference "#PWR052")
@@
 		)
 		(instances
-			(project "wingcam_ee"
+			(project "4reel_ee"
 				(path "/6672ba93-cf23-43d1-a630-d60a05df29bc/45ac4961-8d3d-4c84-aa6c-b96cc3397d34"
 					(reference "C55")
@@
 		)
 		(instances
-			(project "wingcam_ee"
+			(project "4reel_ee"
 				(path "/6672ba93-cf23-43d1-a630-d60a05df29bc/45ac4961-8d3d-4c84-aa6c-b96cc3397d34"
 					(reference "L6")
@@
 		)
 		(instances
-			(project "wingcam_ee"
+			(project "4reel_ee"
 				(path "/6672ba93-cf23-43d1-a630-d60a05df29bc/45ac4961-8d3d-4c84-aa6c-b96cc3397d34"
 					(reference "#PWR094")
@@
 		)
 		(instances
-			(project "wingcam_ee"
+			(project "4reel_ee"
 				(path "/6672ba93-cf23-43d1-a630-d60a05df29bc/45ac4961-8d3d-4c84-aa6c-b96cc3397d34"
 					(reference "#PWR047")
@@
 		)
 		(instances
-			(project "wingcam_ee"
+			(project "4reel_ee"
 				(path "/6672ba93-cf23-43d1-a630-d60a05df29bc/45ac4961-8d3d-4c84-aa6c-b96cc3397d34"
 					(reference "C39")
@@
 		)
 		(instances
-			(project "wingcam_ee"
+			(project "4reel_ee"
 				(path "/6672ba93-cf23-43d1-a630-d60a05df29bc/45ac4961-8d3d-4c84-aa6c-b96cc3397d34"
 					(reference "#PWR095")
@@
 		)
 		(instances
-			(project "wingcam_ee"
+			(project "4reel_ee"
 				(path "/6672ba93-cf23-43d1-a630-d60a05df29bc/45ac4961-8d3d-4c84-aa6c-b96cc3397d34"
 					(reference "C41")
@@
 		)
 		(instances
-			(project "wingcam_ee"
+			(project "4reel_ee"
 				(path "/6672ba93-cf23-43d1-a630-d60a05df29bc/45ac4961-8d3d-4c84-aa6c-b96cc3397d34"
 					(reference "#PWR055")
@@
 		)
 		(instances
-			(project "wingcam_ee"
+			(project "4reel_ee"
 				(path "/6672ba93-cf23-43d1-a630-d60a05df29bc/45ac4961-8d3d-4c84-aa6c-b96cc3397d34"
 					(reference "C51")
@@
 	)
 	(symbol
-		(lib_id "wingcam:OV9281")
+		(lib_id "4reel:OV9281")
 		(at 129.54 35.56 0)
 		(unit 1)
@@
 		)
 		(instances
-			(project "wingcam_ee"
+			(project "4reel_ee"
 				(path "/6672ba93-cf23-43d1-a630-d60a05df29bc/45ac4961-8d3d-4c84-aa6c-b96cc3397d34"
 					(reference "U3")
@@
 		)
 		(instances
-			(project "wingcam_ee"
+			(project "4reel_ee"
 				(path "/6672ba93-cf23-43d1-a630-d60a05df29bc/45ac4961-8d3d-4c84-aa6c-b96cc3397d34"
 					(reference "#PWR096")
@@
 		)
 		(instances
-			(project "wingcam_ee"
+			(project "4reel_ee"
 				(path "/6672ba93-cf23-43d1-a630-d60a05df29bc/45ac4961-8d3d-4c84-aa6c-b96cc3397d34"
 					(reference "#PWR059")
@@
 		)
 		(instances
-			(project "wingcam_ee"
+			(project "4reel_ee"
 				(path "/6672ba93-cf23-43d1-a630-d60a05df29bc/45ac4961-8d3d-4c84-aa6c-b96cc3397d34"
 					(reference "#PWR049")
@@
 		)
 		(instances
-			(project "wingcam_ee"
+			(project "4reel_ee"
 				(path "/6672ba93-cf23-43d1-a630-d60a05df29bc/45ac4961-8d3d-4c84-aa6c-b96cc3397d34"
 					(reference "#PWR045")
@@
 		)
 		(instances
-			(project "wingcam_ee"
+			(project "4reel_ee"
 				(path "/6672ba93-cf23-43d1-a630-d60a05df29bc/45ac4961-8d3d-4c84-aa6c-b96cc3397d34"
 					(reference "#PWR060")
@@
 		)
 		(instances
-			(project "wingcam_ee"
+			(project "4reel_ee"
 				(path "/6672ba93-cf23-43d1-a630-d60a05df29bc/45ac4961-8d3d-4c84-aa6c-b96cc3397d34"
 					(reference "#PWR046")
@@
 		)
 		(instances
-			(project "wingcam_ee"
+			(project "4reel_ee"
 				(path "/6672ba93-cf23-43d1-a630-d60a05df29bc/45ac4961-8d3d-4c84-aa6c-b96cc3397d34"
 					(reference "L4")
@@
 		)
 		(instances
-			(project "wingcam_ee"
+			(project "4reel_ee"
 				(path "/6672ba93-cf23-43d1-a630-d60a05df29bc/45ac4961-8d3d-4c84-aa6c-b96cc3397d34"
 					(reference "R13")
@@
 		)
 		(instances
-			(project "wingcam_ee"
+			(project "4reel_ee"
 				(path "/6672ba93-cf23-43d1-a630-d60a05df29bc/45ac4961-8d3d-4c84-aa6c-b96cc3397d34"
 					(reference "C37")
@@
 		)
 		(instances
-			(project "wingcam_ee"
+			(project "4reel_ee"
 				(path "/6672ba93-cf23-43d1-a630-d60a05df29bc/45ac4961-8d3d-4c84-aa6c-b96cc3397d34"
 					(reference "C52")

Commit message: Worked on the routing.
Changed lines of the file:
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@@
 	(paper "A4")
+	(junction
+		(at 118.11 74.93)
+		(diameter 0)
+		(color 0 0 0 0)
+	)
 	(junction
 		(at 80.01 55.88)
@@
 	(wire
 		(pts
+			(xy 118.11 72.39) (xy 118.11 74.93)
+		)
+		(stroke
+			(width 0)
+			(type default)
+		)
+	)
+	(wire
+		(pts
 			(xy 100.33 63.5) (xy 100.33 64.77)
 		)
@@
 	(wire
 		(pts
-			(xy 111.76 74.93) (xy 129.54 74.93)
+			(xy 111.76 74.93) (xy 118.11 74.93)
 		)
 		(stroke
@@
 		(pts
 			(xy 109.22 119.38) (xy 109.22 120.65)
+		)
+		(stroke
+			(width 0)
+			(type default)
+		)
+	)
+	(wire
+		(pts
+			(xy 118.11 74.93) (xy 129.54 74.93)
 		)
 		(stroke
@@
 		(effects
 			(font
+				(size 1.27 1.27)
+			)
+			(justify left)
+		)
+	)
+	(hierarchical_label "DVDD"
+		(shape bidirectional)
+		(at 118.11 72.39 90)
+		(effects
+			(font

Commit message: R0.1-rc1
Parts:
- C35, C39, C40, C43, C44, C46, C47, C48, C55: MPN (none) -> C0402C105K9PACTU
- C36, C37, C41, C42, C45, C51, C52, C53: MPN (none) -> CL05B104KP5VPNC
- R13: MPN (none) -> RC0402FR-070RL
Changed lines of the file:
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@@
 			)
 		)
+		(property "MPN" "C0402C105K9PACTU"
+			(at 125.73 99.06 0)
+			(hide yes)
+			(show_name no)
+			(do_not_autoplace no)
+			(effects
+				(font
+					(size 1.27 1.27)
+				)
+			)
+		)
 		(pin "1"
 		)
@@
 			)
 		)
+		(property "MPN" "C0402C105K9PACTU"
+			(at 90.17 41.91 0)
+			(hide yes)
+			(show_name no)
+			(do_not_autoplace no)
+			(effects
+				(font
+					(size 1.27 1.27)
+				)
+			)
+		)
 		(pin "1"
 		)
@@
 			)
 		)
+		(property "MPN" "C0402C105K9PACTU"
+			(at 109.22 142.24 0)
+			(hide yes)
+			(show_name no)
+			(do_not_autoplace no)
+			(effects
+				(font
+					(size 1.27 1.27)
+				)
+			)
+		)
 		(pin "1"
 		)
@@
 			)
 		)
+		(property "MPN" "C0402C105K9PACTU"
+			(at 120.65 142.24 0)
+			(hide yes)
+			(show_name no)
+			(do_not_autoplace no)
+			(effects
+				(font
+					(size 1.27 1.27)
+				)
+			)
+		)
 		(pin "1"
 		)
@@
 			)
 		)
+		(property "MPN" "CL05B104KP5VPNC"
+			(at 111.76 41.91 0)
+			(hide yes)
+			(show_name no)
+			(do_not_autoplace no)
+			(effects
+				(font
+					(size 1.27 1.27)
+				)
+			)
+		)
 		(pin "1"
 		)
@@
 			)
 		)
+		(property "MPN" "C0402C105K9PACTU"
+			(at 99.06 142.24 0)
+			(hide yes)
+			(show_name no)
+			(do_not_autoplace no)
+			(effects
+				(font
+					(size 1.27 1.27)
+				)
+			)
+		)
 		(pin "1"
 		)
@@
 			)
 		)
+		(property "MPN" "CL05B104KP5VPNC"
+			(at 124.46 116.84 0)
+			(hide yes)
+			(show_name no)
+			(do_not_autoplace no)
+			(effects
+				(font
+					(size 1.27 1.27)
+				)
+			)
+		)
 		(pin "1"
 		)
@@
 			)
 		)
+		(property "MPN" "C0402C105K9PACTU"
+			(at 90.17 60.96 0)
+			(hide yes)
+			(show_name no)
+			(do_not_autoplace no)
+			(effects
+				(font
+					(size 1.27 1.27)
+				)
+			)
+		)
 		(pin "1"
 		)
@@
 			)
 		)
+		(property "MPN" "CL05B104KP5VPNC"
+			(at 100.33 41.91 0)
+			(hide yes)
+			(show_name no)
+			(do_not_autoplace no)
+			(effects
+				(font
+					(size 1.27 1.27)
+				)
+			)
+		)
 		(pin "1"
 		)
@@
 			)
 		)
+		(property "MPN" "C0402C105K9PACTU"
+			(at 109.22 116.84 0)
+			(hide yes)
+			(show_name no)
+			(do_not_autoplace no)
+			(effects
+				(font
+					(size 1.27 1.27)
+				)
+			)
+		)
 		(pin "1"
 		)
@@
 			)
 		)
+		(property "MPN" "CL05B104KP5VPNC"
+			(at 100.33 60.96 0)
+			(hide yes)
+			(show_name no)
+			(do_not_autoplace no)
+			(effects
+				(font
+					(size 1.27 1.27)
+				)
+			)
+		)
 		(pin "1"
 		)
@@
 			)
 		)
+		(property "MPN" "C0402C105K9PACTU"
+			(at 80.01 60.96 0)
+			(hide yes)
+			(show_name no)
+			(do_not_autoplace no)
+			(effects
+				(font
+					(size 1.27 1.27)
+				)
+			)
+		)
 		(pin "1"
 		)
@@
 			)
 		)
+		(property "MPN" "C0402C105K9PACTU"
+			(at 90.17 80.01 0)
+			(hide yes)
+			(show_name no)
+			(do_not_autoplace no)
+			(effects
+				(font
+					(size 1.27 1.27)
+				)
+			)
+		)
 		(pin "1"
 		)
@@
 			)
 		)
+		(property "MPN" "CL05B104KP5VPNC"
+			(at 100.33 80.01 0)
+			(hide yes)
+			(show_name no)
+			(do_not_autoplace no)
+			(effects
+				(font
+					(size 1.27 1.27)
+				)
+			)
+		)
 		(pin "1"
 		)
@@
 			)
 		)
+		(property "MPN" "CL05B104KP5VPNC"
+			(at 111.76 80.01 0)
+			(hide yes)
+			(show_name no)
+			(do_not_autoplace no)
+			(effects
+				(font
+					(size 1.27 1.27)
+				)
+			)
+		)
 		(pin "1"
 		)
@@
 			)
 		)
+		(property "MPN" "RC0402FR-070RL"
+			(at 116.84 111.76 90)
+			(hide yes)
+			(show_name no)
+			(do_not_autoplace no)
+			(effects
+				(font
+					(size 1.27 1.27)
+				)
+			)
+		)
 		(pin "1"
 		)
@@
 			)
 		)
+		(property "MPN" "CL05B104KP5VPNC"
+			(at 228.6 73.66 0)
+			(hide yes)
+			(show_name no)
+			(do_not_autoplace no)
+			(effects
+				(font
+					(size 1.27 1.27)
+				)
+			)
+		)
 		(pin "1"
 		)
@@
 			(at 111.76 60.96 0)
 			(hide yes)
+			(show_name no)
+			(do_not_autoplace no)
+			(effects
+				(font
+					(size 1.27 1.27)
+				)
+			)
+		)
+		(property "MPN" "CL05B104KP5VPNC"
+			(at 111.76 60.96 0)
+			(hide yes)

Commit message: R0.1 release.
Parts:
- Y1: MPN 7C-24.000MDB-T -> SX5M24.000D20F30TNN
Connections:
- net DOVDD: now also C39.1, C41.1, C51.1, L6.2, U3.B7 (DOVDD), U3.D3 (DOVDD), U3.H2 (DOVDD), U3.H6 (DOVDD); no longer C35.1, C36.1, C52.1, C55.1, L5.2, U3.A2 (DVDD), U3.B1 (DVDD), U3.B3 (DVDD), U3.C5 (DVDD), U3.D8 (DVDD), U3.F2 (DVDD), U3.F3 (EVDD), U3.G1 (DVDD), U3.G6 (DVDD), U3.H5 (EVDD)
- net DVDD: now also C35.1, C36.1, C52.1, C55.1, L5.2, U3.A2 (DVDD), U3.B1 (DVDD), U3.B3 (DVDD), U3.C5 (DVDD), U3.D8 (DVDD), U3.F2 (DVDD), U3.F3 (EVDD), U3.G1 (DVDD), U3.G6 (DVDD), U3.H5 (EVDD); no longer C39.1, C41.1, C51.1, L6.2, U3.B7 (DOVDD), U3.D3 (DOVDD), U3.H2 (DOVDD), U3.H6 (DOVDD)
Changed lines of the file:
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@@
 		)
 	)
-	(label "DOVDD"
+	(label "DVDD"
 		(at 127 55.88 180)
 		(effects
@@
 		)
 	)
-	(label "DVDD"
+	(label "DOVDD"
 		(at 127 74.93 180)
 		(effects
@@
 		)
 	)
-	(hierarchical_label "DVDD"
+	(hierarchical_label "DOVDD"
 		(shape bidirectional)
 		(at 118.11 72.39 90)
@@
 			)
 		)
-		(property "MPN" "7C-24.000MDB-T"
+		(property "MPN" "SX5M24.000D20F30TNN"
 			(at 213.36 78.74 0)
 			(hide yes)

Commit message: Initial schematic, routing finished for RV1106 based design.
Other:
- moved on the sheet: L4, L6
Changed lines of the file:
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@@
 	)
 	(junction
+		(at 111.76 74.93)
+		(diameter 0)
+		(color 0 0 0 0)
+	)
+	(junction
 		(at 90.17 36.83)
 		(diameter 0)
@@
 	)
 	(junction
-		(at 111.76 74.93)
+		(at 90.17 74.93)
 		(diameter 0)
 		(color 0 0 0 0)
@@
 	)
 	(junction
-		(at 90.17 74.93)
-		(diameter 0)
-		(color 0 0 0 0)
-	)
-	(junction
 		(at 124.46 111.76)
 		(diameter 0)
@@
 	(wire
 		(pts
-			(xy 62.23 36.83) (xy 77.47 36.83)
+			(xy 52.07 36.83) (xy 67.31 36.83)
 		)
 		(stroke
@@
 	(wire
 		(pts
-			(xy 62.23 74.93) (xy 77.47 74.93)
+			(xy 52.07 74.93) (xy 67.31 74.93)
 		)
 		(stroke
@@
 	(wire
 		(pts
-			(xy 82.55 74.93) (xy 90.17 74.93)
+			(xy 72.39 74.93) (xy 90.17 74.93)
 		)
 		(stroke
@@
 	(wire
 		(pts
-			(xy 62.23 71.12) (xy 62.23 74.93)
+			(xy 52.07 71.12) (xy 52.07 74.93)
 		)
 		(stroke
@@
 	(wire
 		(pts
-			(xy 82.55 36.83) (xy 90.17 36.83)
+			(xy 72.39 36.83) (xy 90.17 36.83)
 		)
 		(stroke
@@
 	(wire
 		(pts
-			(xy 62.23 33.02) (xy 62.23 36.83)
+			(xy 52.07 33.02) (xy 52.07 36.83)
 		)
 		(stroke
@@
 	(symbol
 		(lib_id "Device:L_Small")
-		(at 80.01 74.93 90)
+		(at 69.85 74.93 90)
 		(unit 1)
 		(body_style 1)
@@
 		(fields_autoplaced yes)
 		(property "Reference" "L6"
-			(at 80.01 69.85 90)
+			(at 69.85 69.85 90)
 			(show_name no)
 			(do_not_autoplace no)
@@
 		)
 		(property "Value" "3u3/0.9A"
-			(at 80.01 72.39 90)
+			(at 69.85 72.39 90)
 			(show_name no)
 			(do_not_autoplace no)
@@
 		)
 		(property "Footprint" "Inductor_SMD:L_0805_2012Metric"
-			(at 80.01 74.93 0)
+			(at 69.85 74.93 0)
 			(hide yes)
 			(show_name no)
@@
 		)
 		(property "Datasheet" ""
-			(at 80.01 74.93 0)
+			(at 69.85 74.93 0)
 			(hide yes)
 			(show_name no)
@@
 		)
 		(property "Description" "Inductor, small symbol"
-			(at 80.01 74.93 0)
+			(at 69.85 74.93 0)
 			(hide yes)
 			(show_name no)
@@
 		)
 		(property "MPN" "MLP2012S3R3MT0S1"
-			(at 80.01 74.93 90)
+			(at 69.85 74.93 90)
 			(hide yes)
 			(show_name no)
@@
 	(symbol
 		(lib_id "power:+5V")
-		(at 62.23 33.02 0)
+		(at 52.07 33.02 0)
 		(unit 1)
 		(body_style 1)
@@
 		(fields_autoplaced yes)
 		(property "Reference" "#PWR047"
-			(at 62.23 36.83 0)
+			(at 52.07 36.83 0)
 			(hide yes)
 			(show_name no)
@@
 		)
 		(property "Value" "+2V8"
-			(at 62.23 27.94 0)
+			(at 52.07 27.94 0)
 			(show_name no)
 			(do_not_autoplace no)
@@
 		)
 		(property "Footprint" ""
-			(at 62.23 33.02 0)
+			(at 52.07 33.02 0)
 			(hide yes)
 			(show_name no)
@@
 		)
 		(property "Datasheet" ""
-			(at 62.23 33.02 0)
+			(at 52.07 33.02 0)
 			(hide yes)
 			(show_name no)
@@
 		)
 		(property "Description" "Power symbol creates a global label with name \"+5V\""
-			(at 62.23 33.02 0)
+			(at 52.07 33.02 0)
 			(hide yes)
 			(show_name no)
@@
 	(symbol
 		(lib_id "power:+5V")
-		(at 62.23 71.12 0)
+		(at 52.07 71.12 0)
 		(unit 1)
 		(body_style 1)
@@
 		(fields_autoplaced yes)
 		(property "Reference" "#PWR046"
-			(at 62.23 74.93 0)
+			(at 52.07 74.93 0)
 			(hide yes)
 			(show_name no)
@@
 		)
 		(property "Value" "+1V8"
-			(at 62.23 66.04 0)
+			(at 52.07 66.04 0)
 			(show_name no)
 			(do_not_autoplace no)
@@
 		)
 		(property "Footprint" ""
-			(at 62.23 71.12 0)
+			(at 52.07 71.12 0)
 			(hide yes)
 			(show_name no)
@@
 		)
 		(property "Datasheet" ""
-			(at 62.23 71.12 0)
+			(at 52.07 71.12 0)
 			(hide yes)
 			(show_name no)
@@
 		)
 		(property "Description" "Power symbol creates a global label with name \"+5V\""
-			(at 62.23 71.12 0)
+			(at 52.07 71.12 0)
 			(hide yes)
 			(show_name no)
@@
 	(symbol
 		(lib_id "Device:L_Small")
-		(at 80.01 36.83 90)
+		(at 69.85 36.83 90)
 		(unit 1)
 		(body_style 1)
@@
 		(fields_autoplaced yes)
 		(property "Reference" "L4"
-			(at 80.01 31.75 90)
+			(at 69.85 31.75 90)
 			(show_name no)
 			(do_not_autoplace no)
@@
 		)
 		(property "Value" "3u3/0.9A"
-			(at 80.01 34.29 90)
+			(at 69.85 34.29 90)
 			(show_name no)
 			(do_not_autoplace no)
@@
 		)
 		(property "Footprint" "Inductor_SMD:L_0805_2012Metric"
-			(at 80.01 36.83 0)
+			(at 69.85 36.83 0)
 			(hide yes)
 			(show_name no)
@@
 		)
 		(property "Datasheet" ""
-			(at 80.01 36.83 0)
+			(at 69.85 36.83 0)
 			(hide yes)
 			(show_name no)
@@
 		)
 		(property "Description" "Inductor, small symbol"
-			(at 80.01 36.83 0)
+			(at 69.85 36.83 0)
 			(hide yes)
 			(show_name no)
@@
 		)
 		(property "MPN" "MLP2012S3R3MT0S1"
-			(at 80.01 36.83 90)
+			(at 69.85 36.83 90)
 			(hide yes)
 			(show_name no)
