File: rv1103/flash.kicad_sch (KiCad schematic)
At the start: 2 parts, among them U7 W25Q32JVZP

Commit message: R0.2 rc
Parts:
- U7: value W25Q32JVZP -> GD25Q128EWIGY; MPN W25Q32JVZPIQ -> GD25Q128EWIGY
Changed lines of the file:
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@@
 			)
 		)
-		(property "Value" "W25Q32JVZP"
+		(property "Value" "GD25Q128EWIGY"
 			(at 162.56 93.9799 0)
 			(show_name no)
@@
 			)
 		)
-		(property "MPN" "W25Q32JVZPIQ"
+		(property "MPN" "GD25Q128EWIGY"
 			(at 151.13 92.71 0)
 			(hide yes)
