File: rv1103/mpu.kicad_sch (KiCad schematic)
At the start: 38 parts, among them U1 RV1103G, Y2 24Mhz

Commit message: Changed LED resistors size and thicken up 0.9V trace.
Parts:
- R23, R24: value 1k -> 470R; MPN RC0402FR-071KL -> RC0402FR-07470RL
Changed lines of the file:
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@@
 			)
 		)
-		(property "Value" "1k"
+		(property "Value" "470R"
 			(at 39.37 128.2699 0)
 			(show_name no)
@@
 			)
 		)
-		(property "MPN" "RC0402FR-071KL"
+		(property "MPN" "RC0402FR-07470RL"
 			(at 36.83 127 0)
 			(hide yes)
@@
 			)
 		)
-		(property "Value" "1k"
+		(property "Value" "470R"
 			(at 27.94 128.2699 0)
 			(show_name no)
@@
 			)
 		)
-		(property "MPN" "RC0402FR-071KL"
+		(property "MPN" "RC0402FR-07470RL"
 			(at 25.4 127 0)
 			(hide yes)

Commit message: R0.2 rc
Parts:
- U1: MPN RV1103BG3 -> RV1103G1
Changed lines of the file:
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@@
 			)
 		)
-		(property "MPN" "RV1103BG3"
+		(property "MPN" "RV1103G1"
 			(at 118.11 146.05 0)
 			(hide yes)
@@
 			)
 		)
-		(property "MPN" "RV1103BG3"
+		(property "MPN" "RV1103G1"
 			(at 219.71 59.69 0)
 			(hide yes)
@@
 			)
 		)
-		(property "MPN" "RV1103BG3"
+		(property "MPN" "RV1103G1"
 			(at 77.47 63.5 0)
 			(hide yes)
